File: Dog Fountain.sch (EAGLE design)
At the start: 19 parts, among them IC1 L298, J1 22-27-2021-02, J4 22-27-2021-02

Commit message: PCB board first test
Parts:
- D1, D2, D3, D4: device diode:DIODE-DO41-10 -> diode:1N5818-B
- R1, R3: value (none) -> 100 Ω
- R2: value (none) -> 180 Ω
Connections:
- net N$11: now also U$1.D7; no longer U$1.D13
- net N$12: now also U$1.D6; no longer U$1.D8
- net N$13: now also U$1.D5; no longer U$1.D7
- net N$14: now also U$1.A5; no longer U$1.D9
- net N$15: now also U$1.A4; no longer U$1.D10
- net N$16: now also U$1.A3; no longer U$1.D11
- net N$5: now also U$1.D2; no longer U$1.D4
- net N$8: now also U$1.D4; no longer U$1.D2
Other:
- moved on the sheet: C1, C2, D5, IC1, J1-1, J1-2, JP4, JP5, R1, R2, R3

Commit message: Another try with 12v power supply
Parts:
- removed B3, B4: RECTIFIER-2KBP, rectifier:RECTIFIER-2KBP
- removed DC1: R-78C5.0-1.0, dc-dc-converter:R-78C5.0-1.0
- removed J4: 22-27-2021-02, con-molex:22-27-2021-02
- added J2: 22-27-2021-02, con-molex:22-27-2021-02
Connections:
- removed net +24V: B4.+, C2.1, D1.C, D2.C, IC1.VS
- removed net N$10: B3.AC2, B4.AC2, J4-1.S
- removed net N$3: B3.+, DC1.VIN
- removed net N$9: B3.AC1, B4.AC1, J4-2.S
- new net +12V: C2.1, D1.C, D2.C, IC1.VS, J2-2.S, U$1.VIN
- net +5V: no longer DC1.VOUT
- net GND: now also J2-1.S; no longer B3.-, B4.-, DC1.GND, IC1.ENABLE_B, IC1.INPUT3, IC1.INPUT4
- net N$4: now also IC1.ENABLE_B
- net N$5: now also IC1.INPUT4
- net N$6: now also IC1.OUT3
- net N$7: now also IC1.OUT4
- net N$8: now also IC1.INPUT3
